Commit message: feat: 3D waiter robot model, doorway path planning & obstacle avoidance, and physical Li-ion battery simulation

File: ros2_ws/src/cstam_gazebo/urdf/cstam_robot.urdf.xacro (robot description, xacro)
@@ -1,16 +1,19 @@
 <?xml version="1.0"?>
-<robot name="cstam_robot" xmlns:xacro="http://www.ros.org/wiki/xacro">
-  <!-- Color Materials -->
-  <material name="cstam_blue">
-    <color rgba="0.1 0.4 0.8 1.0"/>
+<robot name="cstam_waiter_robot" xmlns:xacro="http://www.ros.org/wiki/xacro">
+  <!-- Materials for RViz & Classic Fallback -->
+  <material name="chassis_white">
+    <color rgba="0.92 0.94 0.96 1.0"/>
   </material>
-  <material name="cstam_dark">
-    <color rgba="0.15 0.15 0.18 1.0"/>
+  <material name="metallic_dark">
+    <color rgba="0.15 0.17 0.20 1.0"/>
   </material>
-  <material name="cstam_accent">
-    <color rgba="0.0 0.8 0.7 1.0"/>
+  <material name="accent_cyan">
+    <color rgba="0.0 0.75 0.85 1.0"/>
   </material>
-  <material name="cstam_black">
-    <color rgba="0.05 0.05 0.05 1.0"/>
+  <material name="tray_mat">
+    <color rgba="0.22 0.25 0.28 1.0"/>
+  </material>
+  <material name="screen_glass">
+    <color rgba="0.05 0.08 0.12 1.0"/>
   </material>
   <!-- Base Footprint -->
@@ -19,45 +22,54 @@
     <parent link="base_footprint"/>
     <child link="base_link"/>
-    <origin xyz="0 0 0.1" rpy="0 0 0"/>
-  </joint>
-  <!-- Base Link (Cylindrical Body) -->
+    <origin xyz="0 0 0.09" rpy="0 0 0"/>
+  </joint>
+  <!-- Base Chassis Link -->
   <link name="base_link">
-    <visual>
-      <origin xyz="0 0 0.15" rpy="0 0 0"/>
-      <geometry>
-        <cylinder radius="0.25" length="0.30"/>
-      </geometry>
-      <material name="cstam_blue"/>
-    </visual>
-    <collision>
-      <origin xyz="0 0 0.15" rpy="0 0 0"/>
-      <geometry>
-        <cylinder radius="0.25" length="0.30"/>
-      </geometry>
-    </collision>
-    <inertial>
-      <origin xyz="0 0 0.15" rpy="0 0 0"/>
-      <mass value="15.0"/>
-      <inertia ixx="0.346" ixy="0.0" ixz="0.0" iyy="0.346" iyz="0.0" izz="0.468"/>
-    </inertial>
-  </link>
-  <!-- Left Wheel -->
+    <!-- Main Lower Chassis -->
+    <visual>
+      <origin xyz="0 0 0.08" rpy="0 0 0"/>
+      <geometry>
+        <cylinder radius="0.26" length="0.16"/>
+      </geometry>
+      <material name="chassis_white"/>
+    </visual>
+    <!-- Bumper Ring -->
+    <visual>
+      <origin xyz="0 0 0.02" rpy="0 0 0"/>
+      <geometry>
+        <cylinder radius="0.265" length="0.04"/>
+      </geometry>
+      <material name="metallic_dark"/>
+    </visual>
+    <collision>
+      <origin xyz="0 0 0.08" rpy="0 0 0"/>
+      <geometry>
+        <cylinder radius="0.26" length="0.16"/>
+      </geometry>
+    </collision>
+    <inertial>
+      <origin xyz="0 0 0.06" rpy="0 0 0"/>
+      <mass value="18.0"/>
+      <inertia ixx="0.32" ixy="0.0" ixz="0.0" iyy="0.32" iyz="0.0" izz="0.55"/>
+    </inertial>
+  </link>
+  <!-- Left Drive Wheel -->
   <link name="left_wheel">
     <visual>
       <origin xyz="0 0 0" rpy="1.5707963 0 0"/>
       <geometry>
-        <cylinder radius="0.1" length="0.05"/>
-      </geometry>
-      <material name="cstam_dark"/>
+        <cylinder radius="0.09" length="0.045"/>
+      </geometry>
+      <material name="metallic_dark"/>
     </visual>
     <collision>
       <origin xyz="0 0 0" rpy="1.5707963 0 0"/>
       <geometry>
-        <cylinder radius="0.1" length="0.05"/>
+        <cylinder radius="0.09" length="0.045"/>
       </geometry>
     </collision>
     <inertial>
       <mass value="1.5"/>
-      <inertia ixx="0.004" ixy="0.0" ixz="0.0" iyy="0.004" iyz="0.0" izz="0.0075"/>
+      <inertia ixx="0.0033" ixy="0" ixz="0" iyy="0.0033" iyz="0" izz="0.006"/>
     </inertial>
   </link>
@@ -68,22 +80,22 @@
     <axis xyz="0 1 0"/>
   </joint>
-  <!-- Right Wheel -->
+  <!-- Right Drive Wheel -->
   <link name="right_wheel">
     <visual>
       <origin xyz="0 0 0" rpy="1.5707963 0 0"/>
       <geometry>
-        <cylinder radius="0.1" length="0.05"/>
-      </geometry>
-      <material name="cstam_dark"/>
+        <cylinder radius="0.09" length="0.045"/>
+      </geometry>
+      <material name="metallic_dark"/>
     </visual>
     <collision>
       <origin xyz="0 0 0" rpy="1.5707963 0 0"/>
       <geometry>
-        <cylinder radius="0.1" length="0.05"/>
+        <cylinder radius="0.09" length="0.045"/>
       </geometry>
     </collision>
     <inertial>
       <mass value="1.5"/>
-      <inertia ixx="0.004" ixy="0.0" ixz="0.0" iyy="0.004" iyz="0.0" izz="0.0075"/>
+      <inertia ixx="0.0033" ixy="0" ixz="0" iyy="0.0033" iyz="0" izz="0.006"/>
     </inertial>
   </link>
@@ -94,20 +106,16 @@
     <axis xyz="0 1 0"/>
   </joint>
-  <!-- Caster Wheels (Front & Rear) -->
+  <!-- Front Caster -->
   <link name="caster_front">
     <visual>
-      <geometry>
-        <sphere radius="0.05"/>
-      </geometry>
-      <material name="cstam_black"/>
-    </visual>
-    <collision>
-      <geometry>
-        <sphere radius="0.05"/>
-      </geometry>
+      <geometry><sphere radius="0.045"/></geometry>
+      <material name="metallic_dark"/>
+    </visual>
+    <collision>
+      <geometry><sphere radius="0.045"/></geometry>
     </collision>
     <inertial>
       <mass value="0.5"/>
-      <inertia ixx="0.0005" ixy="0" ixz="0" iyy="0.0005" iyz="0" izz="0.0005"/>
+      <inertia ixx="0.0004" ixy="0" ixz="0" iyy="0.0004" iyz="0" izz="0.0004"/>
     </inertial>
   </link>
@@ -115,21 +123,18 @@
     <parent link="base_link"/>
     <child link="caster_front"/>
-    <origin xyz="0.18 0 -0.05" rpy="0 0 0"/>
-  </joint>
+    <origin xyz="0.18 0 -0.045" rpy="0 0 0"/>
+  </joint>
+  <!-- Rear Caster -->
   <link name="caster_rear">
     <visual>
-      <geometry>
-        <sphere radius="0.05"/>
-      </geometry>
-      <material name="cstam_black"/>
-    </visual>
-    <collision>
-      <geometry>
-        <sphere radius="0.05"/>
-      </geometry>
+      <geometry><sphere radius="0.045"/></geometry>
+      <material name="metallic_dark"/>
+    </visual>
+    <collision>
+      <geometry><sphere radius="0.045"/></geometry>
     </collision>
     <inertial>
       <mass value="0.5"/>
-      <inertia ixx="0.0005" ixy="0" ixz="0" iyy="0.0005" iyz="0" izz="0.0005"/>
+      <inertia ixx="0.0004" ixy="0" ixz="0" iyy="0.0004" iyz="0" izz="0.0004"/>
     </inertial>
   </link>
@@ -137,23 +142,23 @@
     <parent link="base_link"/>
     <child link="caster_rear"/>
-    <origin xyz="-0.18 0 -0.05" rpy="0 0 0"/>
-  </joint>
-  <!-- LiDAR Sensor -->
+    <origin xyz="-0.18 0 -0.045" rpy="0 0 0"/>
+  </joint>
+  <!-- Low-Mounted 360 LiDAR Sensor Link -->
   <link name="laser_frame">
     <visual>
       <origin xyz="0 0 0" rpy="0 0 0"/>
       <geometry>
-        <cylinder radius="0.06" length="0.05"/>
-      </geometry>
-      <material name="cstam_accent"/>
-    </visual>
-    <collision>
-      <geometry>
-        <cylinder radius="0.06" length="0.05"/>
-      </geometry>
-    </collision>
-    <inertial>
-      <mass value="0.3"/>
-      <inertia ixx="0.0003" ixy="0" ixz="0" iyy="0.0003" iyz="0" izz="0.0005"/>
+        <cylinder radius="0.05" length="0.04"/>
+      </geometry>
+      <material name="accent_cyan"/>
+    </visual>
+    <collision>
+      <geometry>
+        <cylinder radius="0.05" length="0.04"/>
+      </geometry>
+    </collision>
+    <inertial>
+      <mass value="0.25"/>
+      <inertia ixx="0.0002" ixy="0" ixz="0" iyy="0.0002" iyz="0" izz="0.0003"/>
     </inertial>
   </link>
@@ -161,5 +166,211 @@
     <parent link="base_link"/>
     <child link="laser_frame"/>
-    <origin xyz="0 0 0.325" rpy="0 0 0"/>
+    <origin xyz="0.16 0 0.13" rpy="0 0 0"/>
+  </joint>
+  <!-- Vertical Structural Spine Columns (Dual Back Pillars) -->
+  <link name="vertical_spine">
+    <!-- Left Upright Pillar -->
+    <visual>
+      <origin xyz="-0.12 0.14 0.50" rpy="0 0 0"/>
+      <geometry><cylinder radius="0.022" length="0.90"/></geometry>
+      <material name="metallic_dark"/>
+    </visual>
+    <collision>
+      <origin xyz="-0.12 0.14 0.50" rpy="0 0 0"/>
+      <geometry><cylinder radius="0.022" length="0.90"/></geometry>
+    </collision>
+    <!-- Right Upright Pillar -->
+    <visual>
+      <origin xyz="-0.12 -0.14 0.50" rpy="0 0 0"/>
+      <geometry><cylinder radius="0.022" length="0.90"/></geometry>
+      <material name="metallic_dark"/>
+    </visual>
+    <collision>
+      <origin xyz="-0.12 -0.14 0.50" rpy="0 0 0"/>
+      <geometry><cylinder radius="0.022" length="0.90"/></geometry>
+    </collision>
+    <!-- Rear Spine Fairing / Shell -->
+    <visual>
+      <origin xyz="-0.14 0 0.50" rpy="0 0 0"/>
+      <geometry><box size="0.04 0.32 0.90"/></geometry>
+      <material name="chassis_white"/>
+    </visual>
+    <collision>
+      <origin xyz="-0.14 0 0.50" rpy="0 0 0"/>
+      <geometry><box size="0.04 0.32 0.90"/></geometry>
+    </collision>
+    <inertial>
+      <origin xyz="-0.12 0 0.50" rpy="0 0 0"/>
+      <mass value="3.5"/>
+      <inertia ixx="0.25" ixy="0" ixz="0" iyy="0.25" iyz="0" izz="0.05"/>
+    </inertial>
+  </link>
+  <joint name="vertical_spine_joint" type="fixed">
+    <parent link="base_link"/>
+    <child link="vertical_spine"/>
+    <origin xyz="0 0 0.16" rpy="0 0 0"/>
+  </joint>
+  <!-- Shelf Tier 1 (Lower Food Shelf) -->
+  <link name="shelf_lower">
+    <!-- Tray Board -->
+    <visual>
+      <origin xyz="0.04 0 0" rpy="0 0 0"/>
+      <geometry><box size="0.38 0.38 0.025"/></geometry>
+      <material name="chassis_white"/>
+    </visual>
+    <!-- Non-slip Surface Mat -->
+    <visual>
+      <origin xyz="0.04 0 0.014" rpy="0 0 0"/>
+      <geometry><box size="0.35 0.35 0.004"/></geometry>
+      <material name="tray_mat"/>
+    </visual>
+    <!-- Front Retaining Rim -->
+    <visual>
+      <origin xyz="0.225 0 0.015" rpy="0 0 0"/>
+      <geometry><box size="0.015 0.38 0.03"/></geometry>
+      <material name="accent_cyan"/>
+    </visual>
+    <!-- Left Retaining Rim -->
+    <visual>
+      <origin xyz="0.04 0.185 0.015" rpy="0 0 0"/>
+      <geometry><box size="0.38 0.015 0.03"/></geometry>
+      <material name="accent_cyan"/>
+    </visual>
+    <!-- Right Retaining Rim -->
+    <visual>
+      <origin xyz="0.04 -0.185 0.015" rpy="0 0 0"/>
+      <geometry><box size="0.38 0.015 0.03"/></geometry>
+      <material name="accent_cyan"/>
+    </visual>
+    <collision>
+      <origin xyz="0.04 0 0.01" rpy="0 0 0"/>
+      <geometry><box size="0.38 0.38 0.04"/></geometry>
+    </collision>
+    <inertial>
+      <mass value="1.2"/>
+      <inertia ixx="0.015" ixy="0" ixz="0" iyy="0.015" iyz="0" izz="0.025"/>
+    </inertial>
+  </link>
+  <joint name="shelf_lower_joint" type="fixed">
+    <parent link="base_link"/>
+    <child link="shelf_lower"/>
+    <origin xyz="0 0 0.30" rpy="0 0 0"/>
+  </joint>
+  <!-- Shelf Tier 2 (Middle Food Shelf) -->
+  <link name="shelf_middle">
+    <visual>
+      <origin xyz="0.04 0 0" rpy="0 0 0"/>
+      <geometry><box size="0.38 0.38 0.025"/></geometry>
+      <material name="chassis_white"/>
+    </visual>
+    <visual>
+      <origin xyz="0.04 0 0.014" rpy="0 0 0"/>
+      <geometry><box size="0.35 0.35 0.004"/></geometry>
+      <material name="tray_mat"/>
+    </visual>
+    <visual>
+      <origin xyz="0.225 0 0.015" rpy="0 0 0"/>
+      <geometry><box size="0.015 0.38 0.03"/></geometry>
+      <material name="accent_cyan"/>
+    </visual>
+    <visual>
+      <origin xyz="0.04 0.185 0.015" rpy="0 0 0"/>
+      <geometry><box size="0.38 0.015 0.03"/></geometry>
+      <material name="accent_cyan"/>
+    </visual>
+    <visual>
+      <origin xyz="0.04 -0.185 0.015" rpy="0 0 0"/>
+      <geometry><box size="0.38 0.015 0.03"/></geometry>
+      <material name="accent_cyan"/>
+    </visual>
+    <collision>
+      <origin xyz="0.04 0 0.01" rpy="0 0 0"/>
+      <geometry><box size="0.38 0.38 0.04"/></geometry>
+    </collision>
+    <inertial>
+      <mass value="1.2"/>
+      <inertia ixx="0.015" ixy="0" ixz="0" iyy="0.015" iyz="0" izz="0.025"/>
+    </inertial>
+  </link>
+  <joint name="shelf_middle_joint" type="fixed">
+    <parent link="base_link"/>
+    <child link="shelf_middle"/>
+    <origin xyz="0 0 0.58" rpy="0 0 0"/>
+  </joint>
+  <!-- Shelf Tier 3 (Upper Food Shelf) -->
+  <link name="shelf_upper">
+    <visual>
+      <origin xyz="0.04 0 0" rpy="0 0 0"/>
+      <geometry><box size="0.38 0.38 0.025"/></geometry>
+      <material name="chassis_white"/>
+    </visual>
+    <visual>
+      <origin xyz="0.04 0 0.014" rpy="0 0 0"/>
+      <geometry><box size="0.35 0.35 0.004"/></geometry>
+      <material name="tray_mat"/>
+    </visual>
+    <visual>
+      <origin xyz="0.225 0 0.015" rpy="0 0 0"/>
+      <geometry><box size="0.015 0.38 0.03"/></geometry>
+      <material name="accent_cyan"/>
+    </visual>
+    <visual>
+      <origin xyz="0.04 0.185 0.015" rpy="0 0 0"/>
+      <geometry><box size="0.38 0.015 0.03"/></geometry>
+      <material name="accent_cyan"/>
+    </visual>
+    <visual>
+      <origin xyz="0.04 -0.185 0.015" rpy="0 0 0"/>
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