Commit message: feat: integrate BellaBot 3D model, restaurant world map, 2D dashboard layout, and fix diagnostics
- Integrate bellabot_v2_assembled.stl into cstam_robot.urdf.xacro and Gazebo models
- Adapt 2D simulation dashboard to restaurant.world with 41 dining tables and service corridor
- Add A* corridor path planning on restaurant occupancy grid
- Update launch files with collision-free spawn coordinates (x: -14.0, y: -2.0)
- Resolve IDE type diagnostics in app.py and delivery_task_manager.py
- Modernize FastAPI startup with async lifespan context manager

File: ros2_ws/src/cstam_gazebo/urdf/cstam_robot.urdf.xacro (robot description, xacro)
@@ -1,7 +1,10 @@
 <?xml version="1.0"?>
 <robot name="cstam_waiter_robot" xmlns:xacro="http://www.ros.org/wiki/xacro">
-  <!-- Materials for RViz & Classic Fallback -->
-  <material name="chassis_white">
-    <color rgba="0.92 0.94 0.96 1.0"/>
+  <!-- Configurable Scaling for BellaBot 3D Mesh -->
+  <!-- 0.00762 scales CAD model (169.2cm) to real-life BellaBot 1.29m height and 0.65m width -->
+  <xacro:property name="mesh_scale" value="0.00762 0.00762 0.00762"/>
+  <!-- Materials for RViz & Simulation -->
+  <material name="bellabot_white">
+    <color rgba="0.94 0.95 0.97 1.0"/>
   </material>
   <material name="metallic_dark">
@@ -17,5 +20,5 @@
     <color rgba="0.05 0.08 0.12 1.0"/>
   </material>
-  <!-- Base Footprint -->
+  <!-- Base Footprint (Ground Projection) -->
   <link name="base_footprint"/>
   <joint name="base_footprint_joint" type="fixed">
@@ -24,32 +27,25 @@
     <origin xyz="0 0 0.09" rpy="0 0 0"/>
   </joint>
-  <!-- Base Chassis Link -->
+  <!-- Base Chassis Link with BellaBot 3D Mesh -->
   <link name="base_link">
-    <!-- Main Lower Chassis -->
-    <visual>
-      <origin xyz="0 0 0.08" rpy="0 0 0"/>
-      <geometry>
-        <cylinder radius="0.26" length="0.16"/>
-      </geometry>
-      <material name="chassis_white"/>
-    </visual>
-    <!-- Bumper Ring -->
-    <visual>
-      <origin xyz="0 0 0.02" rpy="0 0 0"/>
-      <geometry>
-        <cylinder radius="0.265" length="0.04"/>
-      </geometry>
-      <material name="metallic_dark"/>
-    </visual>
-    <collision>
-      <origin xyz="0 0 0.08" rpy="0 0 0"/>
-      <geometry>
-        <cylinder radius="0.26" length="0.16"/>
-      </geometry>
-    </collision>
-    <inertial>
-      <origin xyz="0 0 0.06" rpy="0 0 0"/>
-      <mass value="18.0"/>
-      <inertia ixx="0.32" ixy="0.0" ixz="0.0" iyy="0.32" iyz="0.0" izz="0.55"/>
+    <!-- BellaBot Assembled 3D Visual Mesh -->
+    <visual>
+      <origin xyz="0 0 -0.09" rpy="0 0 1.5707963"/>
+      <geometry>
+        <mesh filename="package://cstam_gazebo/models/robot/mesh/bellabot_v2_assembled.stl" scale="${mesh_scale}"/>
+      </geometry>
+      <material name="bellabot_white"/>
+    </visual>
+    <!-- Stable Physics Collision Cylinder -->
+    <collision>
+      <origin xyz="0 0 0.45" rpy="0 0 0"/>
+      <geometry>
+        <cylinder radius="0.28" length="0.90"/>
+      </geometry>
+    </collision>
+    <inertial>
+      <origin xyz="0 0 0.25" rpy="0 0 0"/>
+      <mass value="25.0"/>
+      <inertia ixx="0.55" ixy="0.0" ixz="0.0" iyy="0.55" iyz="0.0" izz="0.65"/>
     </inertial>
   </link>
@@ -106,5 +102,5 @@
     <axis xyz="0 1 0"/>
   </joint>
-  <!-- Front Caster -->
+  <!-- Front Passive Caster -->
   <link name="caster_front">
     <visual>
@@ -125,5 +121,5 @@
     <origin xyz="0.18 0 -0.045" rpy="0 0 0"/>
   </joint>
-  <!-- Rear Caster -->
+  <!-- Rear Passive Caster -->
   <link name="caster_rear">
     <visual>
@@ -144,10 +140,10 @@
     <origin xyz="-0.18 0 -0.045" rpy="0 0 0"/>
   </joint>
-  <!-- Low-Mounted 360 LiDAR Sensor Link -->
+  <!-- 360-degree LiDAR Sensor Frame (Mounted on front bumper) -->
   <link name="laser_frame">
     <visual>
       <origin xyz="0 0 0" rpy="0 0 0"/>
       <geometry>
-        <cylinder radius="0.05" length="0.04"/>
+        <cylinder radius="0.04" length="0.03"/>
       </geometry>
       <material name="accent_cyan"/>
@@ -155,10 +151,10 @@
     <collision>
       <geometry>
-        <cylinder radius="0.05" length="0.04"/>
-      </geometry>
-    </collision>
-    <inertial>
-      <mass value="0.25"/>
-      <inertia ixx="0.0002" ixy="0" ixz="0" iyy="0.0002" iyz="0" izz="0.0003"/>
+        <cylinder radius="0.04" length="0.03"/>
+      </geometry>
+    </collision>
+    <inertial>
+      <mass value="0.2"/>
+      <inertia ixx="0.0001" ixy="0" ixz="0" iyy="0.0001" iyz="0" izz="0.0002"/>
     </inertial>
   </link>
@@ -166,211 +162,31 @@
     <parent link="base_link"/>
     <child link="laser_frame"/>
-    <origin xyz="0.16 0 0.13" rpy="0 0 0"/>
-  </joint>
-  <!-- Vertical Structural Spine Columns (Dual Back Pillars) -->
-  <link name="vertical_spine">
-    <!-- Left Upright Pillar -->
-    <visual>
-      <origin xyz="-0.12 0.14 0.50" rpy="0 0 0"/>
-      <geometry><cylinder radius="0.022" length="0.90"/></geometry>
-      <material name="metallic_dark"/>
-    </visual>
-    <collision>
-      <origin xyz="-0.12 0.14 0.50" rpy="0 0 0"/>
-      <geometry><cylinder radius="0.022" length="0.90"/></geometry>
-    </collision>
-    <!-- Right Upright Pillar -->
-    <visual>
-      <origin xyz="-0.12 -0.14 0.50" rpy="0 0 0"/>
-      <geometry><cylinder radius="0.022" length="0.90"/></geometry>
-      <material name="metallic_dark"/>
-    </visual>
-    <collision>
-      <origin xyz="-0.12 -0.14 0.50" rpy="0 0 0"/>
-      <geometry><cylinder radius="0.022" length="0.90"/></geometry>
-    </collision>
-    <!-- Rear Spine Fairing / Shell -->
-    <visual>
-      <origin xyz="-0.14 0 0.50" rpy="0 0 0"/>
-      <geometry><box size="0.04 0.32 0.90"/></geometry>
-      <material name="chassis_white"/>
-    </visual>
-    <collision>
-      <origin xyz="-0.14 0 0.50" rpy="0 0 0"/>
-      <geometry><box size="0.04 0.32 0.90"/></geometry>
-    </collision>
-    <inertial>
-      <origin xyz="-0.12 0 0.50" rpy="0 0 0"/>
-      <mass value="3.5"/>
-      <inertia ixx="0.25" ixy="0" ixz="0" iyy="0.25" iyz="0" izz="0.05"/>
-    </inertial>
-  </link>
-  <joint name="vertical_spine_joint" type="fixed">
-    <parent link="base_link"/>
-    <child link="vertical_spine"/>
-    <origin xyz="0 0 0.16" rpy="0 0 0"/>
-  </joint>
-  <!-- Shelf Tier 1 (Lower Food Shelf) -->
-  <link name="shelf_lower">
-    <!-- Tray Board -->
-    <visual>
-      <origin xyz="0.04 0 0" rpy="0 0 0"/>
-      <geometry><box size="0.38 0.38 0.025"/></geometry>
-      <material name="chassis_white"/>
-    </visual>
-    <!-- Non-slip Surface Mat -->
-    <visual>
-      <origin xyz="0.04 0 0.014" rpy="0 0 0"/>
-      <geometry><box size="0.35 0.35 0.004"/></geometry>
-      <material name="tray_mat"/>
-    </visual>
-    <!-- Front Retaining Rim -->
-    <visual>
-      <origin xyz="0.225 0 0.015" rpy="0 0 0"/>
-      <geometry><box size="0.015 0.38 0.03"/></geometry>
-      <material name="accent_cyan"/>
-    </visual>
-    <!-- Left Retaining Rim -->
-    <visual>
-      <origin xyz="0.04 0.185 0.015" rpy="0 0 0"/>
-      <geometry><box size="0.38 0.015 0.03"/></geometry>
-      <material name="accent_cyan"/>
-    </visual>
-    <!-- Right Retaining Rim -->
-    <visual>
-      <origin xyz="0.04 -0.185 0.015" rpy="0 0 0"/>
-      <geometry><box size="0.38 0.015 0.03"/></geometry>
-      <material name="accent_cyan"/>
-    </visual>
-    <collision>
-      <origin xyz="0.04 0 0.01" rpy="0 0 0"/>
-      <geometry><box size="0.38 0.38 0.04"/></geometry>
-    </collision>
-    <inertial>
-      <mass value="1.2"/>
-      <inertia ixx="0.015" ixy="0" ixz="0" iyy="0.015" iyz="0" izz="0.025"/>
-    </inertial>
-  </link>
+    <origin xyz="0.22 0 0.10" rpy="0 0 0"/>
+  </joint>
+  <!-- BellaBot Serving Tray Frames (for TF / Task Monitoring) -->
+  <link name="shelf_lower"/>
   <joint name="shelf_lower_joint" type="fixed">
     <parent link="base_link"/>
     <child link="shelf_lower"/>
-    <origin xyz="0 0 0.30" rpy="0 0 0"/>
-  </joint>
-  <!-- Shelf Tier 2 (Middle Food Shelf) -->
-  <link name="shelf_middle">
-    <visual>
-      <origin xyz="0.04 0 0" rpy="0 0 0"/>
-      <geometry><box size="0.38 0.38 0.025"/></geometry>
-      <material name="chassis_white"/>
-    </visual>
-    <visual>
-      <origin xyz="0.04 0 0.014" rpy="0 0 0"/>
-      <geometry><box size="0.35 0.35 0.004"/></geometry>
-      <material name="tray_mat"/>
-    </visual>
-    <visual>
-      <origin xyz="0.225 0 0.015" rpy="0 0 0"/>
-      <geometry><box size="0.015 0.38 0.03"/></geometry>
-      <material name="accent_cyan"/>
-    </visual>
-    <visual>
-      <origin xyz="0.04 0.185 0.015" rpy="0 0 0"/>
-      <geometry><box size="0.38 0.015 0.03"/></geometry>
-      <material name="accent_cyan"/>
-    </visual>
-    <visual>
-      <origin xyz="0.04 -0.185 0.015" rpy="0 0 0"/>
-      <geometry><box size="0.38 0.015 0.03"/></geometry>
-      <material name="accent_cyan"/>
-    </visual>
-    <collision>
-      <origin xyz="0.04 0 0.01" rpy="0 0 0"/>
-      <geometry><box size="0.38 0.38 0.04"/></geometry>
-    </collision>
-    <inertial>
-      <mass value="1.2"/>
-      <inertia ixx="0.015" ixy="0" ixz="0" iyy="0.015" iyz="0" izz="0.025"/>
-    </inertial>
-  </link>
+    <origin xyz="0.02 0 0.32" rpy="0 0 0"/>
+  </joint>
+  <link name="shelf_middle"/>
   <joint name="shelf_middle_joint" type="fixed">
     <parent link="base_link"/>
     <child link="shelf_middle"/>
-    <origin xyz="0 0 0.58" rpy="0 0 0"/>
-  </joint>
-  <!-- Shelf Tier 3 (Upper Food Shelf) -->
-  <link name="shelf_upper">
-    <visual>
-      <origin xyz="0.04 0 0" rpy="0 0 0"/>
-      <geometry><box size="0.38 0.38 0.025"/></geometry>
-      <material name="chassis_white"/>
-    </visual>
-    <visual>
-      <origin xyz="0.04 0 0.014" rpy="0 0 0"/>
-      <geometry><box size="0.35 0.35 0.004"/></geometry>
-      <material name="tray_mat"/>
-    </visual>
-    <visual>
-      <origin xyz="0.225 0 0.015" rpy="0 0 0"/>
-      <geometry><box size="0.015 0.38 0.03"/></geometry>
-      <material name="accent_cyan"/>
-    </visual>
-    <visual>
-      <origin xyz="0.04 0.185 0.015" rpy="0 0 0"/>
-      <geometry><box size="0.38 0.015 0.03"/></geometry>
-      <material name="accent_cyan"/>
-    </visual>
-    <visual>
-      <origin xyz="0.04 -0.185 0.015" rpy="0 0 0"/>
-      <geometry><box size="0.38 0.015 0.03"/></geometry>
-      <material name="accent_cyan"/>
-    </visual>
-    <collision>
-      <origin xyz="0.04 0 0.01" rpy="0 0 0"/>
-      <geometry><box size="0.38 0.38 0.04"/></geometry>
-    </collision>
-    <inertial>
-      <mass value="1.2"/>
-      <inertia ixx="0.015" ixy="0" ixz="0" iyy="0.015" iyz="0" izz="0.025"/>
-    </inertial>
-  </link>
+    <origin xyz="0.02 0 0.60" rpy="0 0 0"/>
+  </joint>
+  <link name="shelf_upper"/>
   <joint name="shelf_upper_joint" type="fixed">
     <parent link="base_link"/>
     <child link="shelf_upper"/>
-    <origin xyz="0 0 0.85" rpy="0 0 0"/>
-  </joint>
-  <!-- Top Interactive Head Console & Screen Unit -->
-  <link name="head_console">
-    <!-- Top Canopy Head Shell -->
-    <visual>
-      <origin xyz="-0.02 0 0.04" rpy="0 0 0"/>
-      <geometry><box size="0.28 0.34 0.10"/></geometry>
-      <material name="chassis_white"/>
-    </visual>
-    <!-- Customer Interactive Touchscreen Display (Angled 35 deg) -->
-    <visual>
-      <origin xyz="0.06 0 0.06" rpy="0 0.61 0"/>
-      <geometry><box size="0.18 0.24 0.015"/></geometry>
-      <material name="screen_glass"/>
-    </visual>
-    <!-- Waiter Eye / Status Light Bar -->
-    <visual>
-      <origin xyz="0.12 0 0.07" rpy="0 0.61 0"/>
-      <geometry><box size="0.01 0.18 0.02"/></geometry>
-      <material name="accent_cyan"/>
-    </visual>
-    <collision>
-      <origin xyz="-0.02 0 0.04" rpy="0 0 0"/>
-      <geometry><box size="0.28 0.34 0.12"/></geometry>
-    </collision>
-    <inertial>
-      <origin xyz="-0.02 0 0.04" rpy="0 0 0"/>
-      <mass value="1.8"/>
-      <inertia ixx="0.02" ixy="0" ixz="0" iyy="0.02" iyz="0" izz="0.03"/>
-    </inertial>
-  </link>
+    <origin xyz="0.02 0 0.88" rpy="0 0 0"/>
+  </joint>
+  <!-- BellaBot Head Console Frame -->
+  <link name="head_console"/>
   <joint name="head_console_joint" type="fixed">
     <parent link="base_link"/>
     <child link="head_console"/>
-    <origin xyz="0 0 1.05" rpy="0 0 0"/>
+    <origin xyz="0.05 0 1.15" rpy="0 0.35 0"/>
   </joint>
   <!-- Gazebo Sim Differential Drive Plugin -->
@@ -415,5 +231,5 @@
         <range>
           <min>0.10</min>
-          <max>12.0</max>
+          <max>15.0</max>
           <resolution>0.015</resolution>
         </range>
@@ -431,41 +247,9 @@
     <visual>
       <material>
-        <ambient>0.92 0.94 0.96 1.0</ambient>
-        <diffuse>0.92 0.94 0.96 1.0</diffuse>
+        <ambient>0.94 0.95 0.97 1.0</ambient>
+        <diffuse>0.94 0.95 0.97 1.0</diffuse>
         <specular>0.4 0.4 0.4 1.0</specular>
       </material>
     </visual>
   </gazebo>
-  <gazebo reference="shelf_lower">
-    <visual>
-      <material>
-        <ambient>0.25 0.28 0.32 1.0</ambient>
-        <diffuse>0.25 0.28 0.32 1.0</diffuse>
-      </material>
-    </visual>
-  </gazebo>
-  <gazebo reference="shelf_middle">
-    <visual>
-      <material>
-        <ambient>0.25 0.28 0.32 1.0</ambient>
-        <diffuse>0.25 0.28 0.32 1.0</diffuse>
-      </material>
-    </visual>
-  </gazebo>
-  <gazebo reference="shelf_upper">
-    <visual>
-      <material>
-        <ambient>0.25 0.28 0.32 1.0</ambient>
-        <diffuse>0.25 0.28 0.32 1.0</diffuse>
-      </material>
-    </visual>
-  </gazebo>
-  <gazebo reference="head_console">
-    <visual>
-      <material>
-        <ambient>0.92 0.94 0.96 1.0</ambient>
-        <diffuse>0.92 0.94 0.96 1.0</diffuse>
-      </material>
-    </visual>
-  </gazebo>
 </robot>

Commit message: Phase 1 only

File: ros2_ws/src/cstam_gazebo/urdf/cstam_robot.urdf.xacro (robot description, xacro)
@@ -41,5 +41,5 @@
       <origin xyz="0 0 0.45" rpy="0 0 0"/>
       <geometry>
-        <cylinder radius="0.28" length="0.90"/>
+        <cylinder radius="0.22" length="0.90"/>
       </geometry>
     </collision>
@@ -162,5 +162,5 @@
     <parent link="base_link"/>
     <child link="laser_frame"/>
-    <origin xyz="0.22 0 0.10" rpy="0 0 0"/>
+    <origin xyz="0.32 0 0.12" rpy="0 0 0"/>
   </joint>
   <!-- BellaBot Serving Tray Frames (for TF / Task Monitoring) -->
@@ -199,6 +199,6 @@
       <max_linear_acceleration>1.2</max_linear_acceleration>
       <max_angular_acceleration>2.5</max_angular_acceleration>
-      <topic>cmd_vel</topic>
-      <odom_topic>odom</odom_topic>
+      <topic>/cmd_vel</topic>
+      <odom_topic>/odom</odom_topic>
       <frame_id>odom</frame_id>
       <child_frame_id>base_footprint</child_frame_id>
@@ -225,10 +225,10 @@
             <samples>360</samples>
             <resolution>1.0</resolution>
-            <min_angle>-3.14159</min_angle>
-            <max_angle>3.14159</max_angle>
+            <min_angle>-2.35619</min_angle>
+            <max_angle>2.35619</max_angle>
           </horizontal>
         </scan>
         <range>
-          <min>0.10</min>
+          <min>0.12</min>
           <max>15.0</max>
           <resolution>0.015</resolution>
@@ -253,3 +253,32 @@
     </visual>
   </gazebo>
+  <!-- Wheel and Caster Friction for Gazebo Sim -->
+  <gazebo reference="left_wheel">
+    <mu1>1.0</mu1>
+    <mu2>1.0</mu2>
+    <kp>1000000.0</kp>
+    <kd>100.0</kd>
+    <minDepth>0.001</minDepth>
+  </gazebo>
+  <gazebo reference="right_wheel">
+    <mu1>1.0</mu1>
+    <mu2>1.0</mu2>
+    <kp>1000000.0</kp>
+    <kd>100.0</kd>
+    <minDepth>0.001</minDepth>
+  </gazebo>
+  <gazebo reference="caster_front">
+    <mu1>0.001</mu1>
+    <mu2>0.001</mu2>
+    <kp>1000000.0</kp>
+    <kd>100.0</kd>
+    <minDepth>0.001</minDepth>
+  </gazebo>
+  <gazebo reference="caster_rear">
+    <mu1>0.001</mu1>
+    <mu2>0.001</mu2>
+    <kp>1000000.0</kp>
+    <kd>100.0</kd>
+    <minDepth>0.001</minDepth>
+  </gazebo>
 </robot>
